File: KES-K5170/KES.kicad_sch (KiCad schematic)
At the start: 94 parts, among them X1 DIN41612_03x32_ABC, X2 DIN41612_03x32_ABC

Commit message: KES - Bugfix: UCC/USS bei einigen Symbolen vertauscht - Bugfix: Leiterbahnen Ober/Unterseite vertauscht
AFS:
- Neu

Symbole:
- verschoben
Parts:
- X1, X2: footprint Connector_DIN:DIN41612_R_3x32_Female_Horizontal_THT -> Connector_DIN:DIN41612_C_3x32_Male_Horizontal_THT
Connections:
- net +5V: now also AEAO1.16 (UCC), AEBK1.16 (UCC), AGCI1.24 (UCC), AKDM1.18 (UCC), AKEI1.18 (UCC), AQAM1.20 (UCC), AQBK1.20 (UCC), ASDM1.18 (UCC), ASEI1.18 (UCC), AWCI1.24 (UCC), BEDM1.18 (UCC), BEEI1.18 (UCC), BMDM1.18 (UCC), BMEI1.18 (UCC), BOBK1.20 (UCC), BOCI1.24 (UCC), BWDM1.18 (UCC), BWEI1.18 (UCC), CGCI1.24 (UCC), CGDM1.18 (UCC), CGEI1.18 (UCC), CQDM1.18 (UCC), CQEI1.18 (UCC), DADM1.18 (UCC), DAEI1.18 (UCC); no longer AEAO1.8 (UCC), AEBK1.8 (UCC), AGCI1.12 (UCC), AKDM1.9 (UCC), AKEI1.9 (UCC), AQAM1.10 (UCC), AQBK1.10 (UCC), ASDM1.9 (UCC), ASEI1.9 (UCC), AWCI1.12 (UCC), BEDM1.9 (UCC), BEEI1.9 (UCC), BMDM1.9 (UCC), BMEI1.9 (UCC), BOBK1.10 (UCC), BOCI1.12 (UCC), BWDM1.9 (UCC), BWEI1.9 (UCC), CGCI1.12 (UCC), CGDM1.9 (UCC), CGEI1.9 (UCC), CQDM1.9 (UCC), CQEI1.9 (UCC), DADM1.9 (UCC), DAEI1.9 (UCC)
- net GND: now also AEAO1.8 (GND), AEBK1.8 (GND), AGCI1.12 (GND), AKDM1.9 (GND), AKEI1.9 (GND), AQAM1.10 (GND), AQBK1.10 (GND), ASDM1.9 (GND), ASEI1.9 (GND), AWCI1.12 (GND), BEDM1.9 (GND), BEEI1.9 (GND), BMDM1.9 (GND), BMEI1.9 (GND), BOBK1.10 (GND), BOCI1.12 (GND), BWDM1.9 (GND), BWEI1.9 (GND), CGCI1.12 (GND), CGDM1.9 (GND), CGEI1.9 (GND), CQDM1.9 (GND), CQEI1.9 (GND), DADM1.9 (GND), DAEI1.9 (GND); no longer AEAO1.16 (GND), AEBK1.16 (GND), AGCI1.24 (GND), AKDM1.18 (GND), AKEI1.18 (GND), AQAM1.20 (GND), AQBK1.20 (GND), ASDM1.18 (GND), ASEI1.18 (GND), AWCI1.24 (GND), BEDM1.18 (GND), BEEI1.18 (GND), BMDM1.18 (GND), BMEI1.18 (GND), BOBK1.20 (GND), BOCI1.24 (GND), BWDM1.18 (GND), BWEI1.18 (GND), CGCI1.24 (GND), CGDM1.18 (GND), CGEI1.18 (GND), CQDM1.18 (GND), CQEI1.18 (GND), DADM1.18 (GND), DAEI1.18 (GND)
Changed lines of the file:
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@@
 			)
 		)
-		(property "Footprint" "Connector_DIN:DIN41612_R_3x32_Female_Horizontal_THT"
+		(property "Footprint" "Connector_DIN:DIN41612_C_3x32_Male_Horizontal_THT"
 			(at 158.75 359.41 0)
 			(effects
@@
 		(pin "2"
 		)
-		(pin "3"
-		)
 		(pin "9"
 		)
@@
 	(symbol
 		(lib_id "Robotron_Symbole:7474")
-		(at 473.71 350.52 0)
-		(mirror x)
+		(at 473.71 346.71 0)
 		(unit 3)
 		(exclude_from_sim no)
@@
 		(dnp no)
 		(property "Reference" "FCDM1"
-			(at 476.504 343.408 0)
+			(at 476.504 353.822 0)
 			(effects
 				(font
@@
 		)
 		(property "Value" "7474"
-			(at 476.504 354.076 0)
+			(at 476.504 343.154 0)
 			(effects
 				(font
@@
 		)
 		(property "Footprint" "Package_DIP:DIP-14_W7.62mm"
-			(at 473.71 350.52 0)
+			(at 473.71 346.71 0)
 			(effects
 				(font
@@
 		)
 		(property "Datasheet" ""
-			(at 473.71 350.52 0)
+			(at 473.71 346.71 0)
 			(effects
 				(font
@@
 		)
 		(property "Description" ""
-			(at 473.71 350.52 0)
+			(at 473.71 346.71 0)
 			(effects
 				(font
@@
 	(symbol
 		(lib_id "Robotron_Symbole:7474")
-		(at 480.06 350.52 0)
-		(mirror x)
+		(at 480.06 346.71 0)
 		(unit 3)
 		(exclude_from_sim no)
@@
 		(dnp no)
 		(property "Reference" "FCEK1"
-			(at 482.854 343.408 0)
+			(at 482.854 353.822 0)
 			(effects
 				(font
@@
 		)
 		(property "Value" "7474"
-			(at 482.854 353.568 0)
+			(at 482.854 343.662 0)
 			(effects
 				(font
@@
 		)
 		(property "Footprint" "Package_DIP:DIP-14_W7.62mm"
-			(at 480.06 350.52 0)
+			(at 480.06 346.71 0)
 			(effects
 				(font
@@
 		)
 		(property "Datasheet" ""
-			(at 480.06 350.52 0)
+			(at 480.06 346.71 0)
 			(effects
 				(font
@@
 		)
 		(property "Description" ""
-			(at 480.06 350.52 0)
+			(at 480.06 346.71 0)
 			(effects
 				(font
@@
 	(symbol
 		(lib_id "Robotron_Symbole:7474")
-		(at 486.41 350.52 0)
-		(mirror x)
+		(at 486.41 346.71 0)
 		(unit 3)
 		(exclude_from_sim no)
@@
 		(dnp no)
 		(property "Reference" "EQCO1"
-			(at 489.204 343.408 0)
+			(at 489.204 353.822 0)
 			(effects
 				(font
@@
 		)
 		(property "Value" "7474"
-			(at 489.458 354.076 0)
+			(at 489.458 343.154 0)
 			(effects
 				(font
@@
 		)
 		(property "Footprint" "Package_DIP:DIP-14_W7.62mm"
-			(at 486.41 350.52 0)
+			(at 486.41 346.71 0)
 			(effects
 				(font
@@
 		)
 		(property "Datasheet" ""
-			(at 486.41 350.52 0)
+			(at 486.41 346.71 0)
 			(effects
 				(font
@@
 		)
 		(property "Description" ""
-			(at 486.41 350.52 0)
+			(at 486.41 346.71 0)
 			(effects
 				(font
@@
 	(symbol
 		(lib_id "Robotron_Symbole:7474")
-		(at 505.46 350.52 0)
-		(mirror x)
+		(at 505.46 346.71 0)
 		(unit 3)
 		(exclude_from_sim no)
@@
 		(dnp no)
 		(property "Reference" "GQAS1"
-			(at 508.508 343.408 0)
+			(at 508.508 353.822 0)
 			(effects
 				(font
@@
 		)
 		(property "Value" "7474"
-			(at 508.508 354.076 0)
+			(at 508.508 343.154 0)
 			(effects
 				(font
@@
 		)
 		(property "Footprint" "Package_DIP:DIP-14_W7.62mm"
-			(at 505.46 350.52 0)
+			(at 505.46 346.71 0)
 			(effects
 				(font
@@
 		)
 		(property "Datasheet" ""
-			(at 505.46 350.52 0)
+			(at 505.46 346.71 0)
 			(effects
 				(font
@@
 		)
 		(property "Description" ""
-			(at 505.46 350.52 0)
+			(at 505.46 346.71 0)
 			(effects
 				(font
@@
 			)
 		)
-		(property "Footprint" "Connector_DIN:DIN41612_R_3x32_Female_Horizontal_THT"
+		(property "Footprint" "Connector_DIN:DIN41612_C_3x32_Male_Horizontal_THT"
 			(at 158.75 396.24 0)
 			(effects
@@
 	(symbol
 		(lib_id "Robotron_Symbole:7474")
-		(at 499.11 350.52 0)
-		(mirror x)
+		(at 499.11 346.71 0)
 		(unit 3)
 		(exclude_from_sim no)
@@
 		(dnp no)
 		(property "Reference" "FMDM1"
-			(at 501.904 343.408 0)
+			(at 501.904 353.822 0)
 			(effects
 				(font
@@
 		)
 		(property "Value" "7474"
-			(at 501.65 354.076 0)
+			(at 501.65 343.154 0)
 			(effects
 				(font
@@
 		)
 		(property "Footprint" "Package_DIP:DIP-14_W7.62mm"
-			(at 499.11 350.52 0)
+			(at 499.11 346.71 0)
 			(effects
 				(font
@@
 		)
 		(property "Datasheet" ""
-			(at 499.11 350.52 0)
+			(at 499.11 346.71 0)
 			(effects
 				(font
@@
 		)
 		(property "Description" ""
-			(at 499.11 350.52 0)
+			(at 499.11 346.71 0)
 			(effects
 				(font
@@
 	(symbol
 		(lib_id "Robotron_Symbole:7474")
-		(at 467.36 350.52 0)
-		(mirror x)
+		(at 467.36 346.71 0)
 		(unit 3)
 		(exclude_from_sim no)
@@
 		(dnp no)
 		(property "Reference" "DUDM1"
-			(at 470.408 343.662 0)
+			(at 470.408 353.568 0)
 			(effects
 				(font
@@
 		)
 		(property "Value" "7474"
-			(at 469.9 354.33 0)
+			(at 469.9 342.9 0)
 			(effects
 				(font
@@
 		)
 		(property "Footprint" "Package_DIP:DIP-14_W7.62mm"
-			(at 467.36 350.52 0)
+			(at 467.36 346.71 0)
 			(effects
 				(font
@@
 		)
 		(property "Datasheet" ""
-			(at 467.36 350.52 0)
+			(at 467.36 346.71 0)
 			(effects
 				(font
@@
 		)
 		(property "Description" ""
-			(at 467.36 350.52 0)
+			(at 467.36 346.71 0)
 			(effects
 				(font
@@
 	(symbol
 		(lib_id "Robotron_Symbole:7474")
-		(at 492.76 350.52 0)
-		(mirror x)
+		(at 492.76 346.71 0)
 		(unit 3)
 		(exclude_from_sim no)
@@
 		(dnp no)
 		(property "Reference" "GIDM1"
-			(at 495.808 343.408 0)
+			(at 495.808 353.822 0)
 			(effects
 				(font
@@
 		)
 		(property "Value" "7474"
-			(at 495.808 353.568 0)
+			(at 495.808 343.662 0)
 			(effects
 				(font
@@
 		)
 		(property "Footprint" "Package_DIP:DIP-14_W7.62mm"
-			(at 492.76 350.52 0)
+			(at 492.76 346.71 0)
 			(effects
 				(font
@@
 		)
 		(property "Datasheet" ""
-			(at 492.76 350.52 0)
+			(at 492.76 346.71 0)
 			(effects
 				(font
@@
 		)
 		(property "Description" ""
-			(at 492.76 350.52 0)
+			(at 492.76 346.71 0)
 			(effects
 				(font
