File: KES-K5170/KES_B2.kicad_sch (KiCad schematic)
At the start: 46 parts, among them J1 Conn_01x01, J10 Conn_01x01, J11 Conn_01x01, J12 Conn_01x01, J16 Conn_01x01, J17 Conn_01x01, J18 Conn_01x01, J19 Conn_01x01, J20 Conn_01x01, J21 Conn_01x01, J22 Conn_01x01, J23 Conn_01x01, J24 Conn_01x01, J3 Conn_01x01, J33 Conn_01x01, J34 Conn_01x01, J35 Conn_01x01, J36 Conn_01x01, J37 Conn_01x01, J38 Conn_01x01, J47 Conn_01x01, J48 Conn_01x01, J49 Conn_01x01, J5 Conn_01x01, J50 Conn_01x01, J51 Conn_01x01, J52 Conn_01x01, J53 Conn_01x01, J54 Conn_01x01, J6 Conn_01x01, J9 Conn_01x01

Commit message: KES - Bugfix: UCC/USS bei einigen Symbolen vertauscht - Bugfix: Leiterbahnen Ober/Unterseite vertauscht
AFS:
- Neu

Symbole:
- verschoben
Connections:
- net +5V: now also BCAM1.20 (UCC), BCBK1.20 (UCC), BOAM1.20 (UCC), FCAM1.20 (UCC), FCCM1.20 (UCC), FMAM1.20 (UCC), FMBM1.20 (UCC), FMCM1.20 (UCC), FWAM1.20 (UCC), FWBM1.20 (UCC), FWCM1.20 (UCC); no longer BCAM1.10 (UCC), BCBK1.10 (UCC), BOAM1.10 (UCC), FCAM1.10 (UCC), FCCM1.10 (UCC), FMAM1.10 (UCC), FMBM1.10 (UCC), FMCM1.10 (UCC), FWAM1.10 (UCC), FWBM1.10 (UCC), FWCM1.10 (UCC)
- net GND: now also BCAM1.10 (GND), BCBK1.10 (GND), BOAM1.10 (GND), FCAM1.10 (GND), FCCM1.10 (GND), FMAM1.10 (GND), FMBM1.10 (GND), FMCM1.10 (GND), FWAM1.10 (GND), FWBM1.10 (GND), FWCM1.10 (GND); no longer BCAM1.20 (GND), BCBK1.20 (GND), BOAM1.20 (GND), FCAM1.20 (GND), FCCM1.20 (GND), FMAM1.20 (GND), FMBM1.20 (GND), FMCM1.20 (GND), FWAM1.20 (GND), FWBM1.20 (GND), FWCM1.20 (GND)
