File: KES-K5170/KES_B3.kicad_sch (KiCad schematic)
At the start: 67 parts, among them X1001 Conn_01x01, X1002 Conn_01x01, X1003 Conn_01x01, X1004 Conn_01x01, X1005 Conn_01x01, X1006 Conn_01x01, X1007 Conn_01x01, X1008 Conn_01x01, X1009 Conn_01x01, X1010 Conn_01x01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

Commit message: KES - Bugfix: UCC/USS bei einigen Symbolen vertauscht - Bugfix: Leiterbahnen Ober/Unterseite vertauscht
AFS:
- Neu

Symbole:
- verschoben
Connections:
- net +5V: now also DUCK1.20 (UCC), GIBO1.16 (UCC), GSEI1.18 (UCC), HEAO1.20 (UCC), HEDM1.16 (UCC); no longer DUCK1.10 (UCC), GIBO1.8 (UCC), GSEI1.10 (UCC), HEAO1.10 (UCC), HEDM1.8 (UCC)
- net GND: now also DUCK1.10 (GND), GIBO1.8 (GND), GSEI1.9 (GND), HEAO1.10 (GND), HEDM1.8 (GND); no longer DUCK1.20 (GND), GIBO1.16 (GND), GSEI1.20 (GND), HEAO1.20 (GND), HEDM1.16 (GND)
Other:
- note added: "Auf der A7100-Variante nicht vorhanden, auf der A7150-Variante mit Lackdrat ausgeführt."
- note removed: "Im original-Stromlaufplan vorhanden, auf Platine nicht geroutet!"
Changed lines of the file:
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@@
 		)
 	)
-	(text "Im original-Stromlaufplan vorhanden,\nauf Platine nicht geroutet!"
+	(text "Auf der A7100-Variante nicht vorhanden,\nauf der A7150-Variante mit Lackdrat ausgeführt."
 		(exclude_from_sim no)
 		(at 547.116 323.596 0)
@@
 		(pin "2"
 		)
-		(pin "3"
-		)
 		(pin "9"
 		)
@@
 	)
 	(symbol
-		(lib_name "7420_1")
 		(lib_id "Robotron_Symbole:7420")
 		(at 287.02 340.36 0)
@@
 		(pin "1"
 		)
-		(pin "20"
+		(pin "18"
 		)
-		(pin "10"
+		(pin "9"
 		)
 		(instances
